File: femu/femu-1.0.3.c_2-LAYER.brd (EAGLE design)
At the start: 44.6 x 21.1 mm, 74 parts, among them IC1 ESP32-QFN_5X5

Commit message: Adding work on femu 1.0.2, and 1.0.3
Parts:
- renumbered U$11 to IC2, U$57 to LDO2
Changed lines of the file:
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@@
 </element>
 <element name="C13" library="parts_0201" package="PART" value="0.1uF" x="29.4894" y="5.7146" smashed="yes" rot="R90">
-<attribute name="MPN" value="GRM022R60G104ME15L" x="54.5394" y="-3.2854" size="0.5" layer="27" rot="R90" display="off"/>
+<attribute name="MPN" value="GRM033R61C104KE84D" x="54.5394" y="-3.2854" size="0.5" layer="27" rot="R90" display="off"/>
 </element>
 <element name="C15" library="parts_0201" package="PART" value="1uF" x="26.035" y="8.636" smashed="yes" rot="R90">
@@
 </element>
 <element name="C23" library="parts_0201" package="PART" value="4.7uF" x="18.161" y="7.239" smashed="yes" rot="R270">
-<attribute name="MPN" value="GRM035R60G475ME15D" x="18.161" y="7.239" size="1.778" layer="27" rot="R270" display="off"/>
+<attribute name="MPN" value="GRM035R60J475ME15D" x="18.161" y="7.239" size="1.778" layer="27" rot="R270" display="off"/>
 </element>
 <element name="C24" library="parts_0201" package="PART" value="10nF" x="13.5128" y="8.001" smashed="yes" rot="R270">
@@
 </element>
 <element name="U$6" library="femu-edge-connectors" package="FEMU-EDGE-CONNECTOR" value="FEMU-EDGE-CONNECTOR" x="37.8968" y="3.8354" smashed="yes"/>
-<element name="U$11" library="ftdi_ft231x" package="QFN-20_4X4" value="FT231XQ" x="17.2974" y="10.7442" smashed="yes" rot="R270">
+<element name="IC2" library="ftdi_ft231x" package="QFN-20_4X4" value="FT231XQ" x="17.2974" y="10.7442" smashed="yes" rot="R270">
 <attribute name="MPN" value="FT231XQ" x="17.2974" y="10.7442" size="1.778" layer="27" rot="R270" display="off"/>
 </element>
@@
 <attribute name="MPN" value="ERJ-1GN0R00C" x="21.7678" y="-2.54" size="1.778" layer="27" display="off"/>
 </element>
-<element name="U$57" library="onsemi" package="WLCSP4_0.65X0.65MM" value="FAN25800AUC33X" x="21.1328" y="2.8194" smashed="yes">
+<element name="LDO2" library="onsemi" package="WLCSP4_0.65X0.65MM" value="FAN25800AUC33X" x="21.1328" y="2.8194" smashed="yes">
 <attribute name="MPN" value="FAN25800AUC33X" x="21.1328" y="2.8194" size="1.778" layer="27" display="off"/>
+<attribute name="MPN_ALT" value="NCP167BFCT330T2G" x="21.1328" y="2.8194" size="1.778" layer="27" display="off"/>
 </element>
 <element name="R16" library="parts_0201" package="PART" value="1K" x="19.939" y="2.54" smashed="yes">
@@
 <contactref element="C2" pad="1"/>
 <contactref element="U$6" pad="1"/>
-<contactref element="U$11" pad="3"/>
-<contactref element="U$11" pad="21"/>
-<contactref element="U$11" pad="13"/>
+<contactref element="IC2" pad="3"/>
+<contactref element="IC2" pad="21"/>
+<contactref element="IC2" pad="13"/>
 <contactref element="U$49" pad="P$1"/>
 <polygon width="0.127" layer="16">
@@
 <wire x1="40.491" y1="17.145" x2="40.491" y2="14.859" width="0.254" layer="1"/>
 <contactref element="R17" pad="1"/>
-<contactref element="U$57" pad="GND"/>
+<contactref element="LDO2" pad="GND"/>
 <wire x1="21.844" y1="3.81" x2="22.733" y2="3.81" width="0.2032" layer="1"/>
 <wire x1="19.05" y1="3.302" x2="19.05" y2="3.9624" width="0.2032" layer="1"/>
@@
 <contactref element="RGB1" pad="1"/>
 <contactref element="U$6" pad="2"/>
-<contactref element="U$11" pad="10"/>
-<contactref element="U$11" pad="11"/>
-<contactref element="U$11" pad="20"/>
+<contactref element="IC2" pad="10"/>
+<contactref element="IC2" pad="11"/>
+<contactref element="IC2" pad="20"/>
 <contactref element="C25" pad="2"/>
 <contactref element="R7" pad="1"/>
@@
 <signal name="TXD">
 <contactref element="IC1" pad="41"/>
-<contactref element="U$11" pad="1"/>
+<contactref element="IC2" pad="1"/>
 <contactref element="U$50" pad="P$2"/>
 <wire x1="25.5534" y1="10.4202" x2="25.5534" y2="9.6784" width="0.1524" layer="1"/>
@@
 <signal name="RXD">
 <contactref element="IC1" pad="40"/>
-<contactref element="U$11" pad="17"/>
+<contactref element="IC2" pad="17"/>
 <contactref element="U$50" pad="P$1"/>
 <wire x1="25.2034" y1="10.4202" x2="25.2034" y2="9.8364" width="0.1524" layer="1"/>
@@
 <wire x1="18.415" y1="4.7244" x2="18.415" y2="6.35" width="0.254" layer="1"/>
 <wire x1="18.415" y1="6.35" x2="18.415" y2="6.762" width="0.254" layer="1"/>
-<contactref element="U$11" pad="12"/>
+<contactref element="IC2" pad="12"/>
 <wire x1="14.732" y1="6.858" x2="14.763" y2="6.889" width="0.254" layer="1"/>
 <wire x1="14.763" y1="6.889" x2="16.764" y2="6.889" width="0.254" layer="1"/>
@@
 <signal name="USB-">
 <contactref element="R8" pad="2"/>
-<contactref element="U$11" pad="9"/>
+<contactref element="IC2" pad="9"/>
 <wire x1="15.4474" y1="10.2442" x2="14.4042" y2="10.2442" width="0.254" layer="1"/>
 <wire x1="14.4042" y1="10.2442" x2="14.193" y2="10.033" width="0.254" layer="1"/>
@@
 <signal name="USB+">
 <contactref element="R9" pad="2"/>
-<contactref element="U$11" pad="8"/>
+<contactref element="IC2" pad="8"/>
 <wire x1="15.4474" y1="10.7442" x2="14.3708" y2="10.7442" width="0.254" layer="1"/>
 <wire x1="14.3708" y1="10.7442" x2="14.193" y2="10.922" width="0.254" layer="1"/>
@@
 <contactref element="C22" pad="2"/>
 <contactref element="R2" pad="2"/>
-<contactref element="U$11" pad="19"/>
+<contactref element="IC2" pad="19"/>
 <contactref element="U$50" pad="P$3"/>
 <wire x1="28.7284" y1="13.2452" x2="29.03539375" y2="13.2452" width="0.1524" layer="1"/>
@@
 <signal name="BOOT/DTR">
 <contactref element="IC1" pad="23"/>
-<contactref element="U$11" pad="18"/>
+<contactref element="IC2" pad="18"/>
 <contactref element="R7" pad="2"/>
 <contactref element="U$51" pad="P$1"/>
@@
 <contactref element="R12" pad="1"/>
 <contactref element="R16" pad="1"/>
-<contactref element="U$57" pad="VIN"/>
+<contactref element="LDO2" pad="VIN"/>
 <wire x1="20.9578" y1="2.9944" x2="20.6502" y2="3.302" width="0.2032" layer="1"/>
 <wire x1="20.6502" y1="3.302" x2="20.066" y2="3.302" width="0.2032" layer="1"/>
@@
 <contactref element="C30" pad="2"/>
 <contactref element="R13" pad="1"/>
-<contactref element="U$57" pad="VOUT"/>
+<contactref element="LDO2" pad="VOUT"/>
 <wire x1="21.3078" y1="3.3302" x2="20.828" y2="3.81" width="0.2032" layer="1"/>
 <wire x1="21.3078" y1="2.9944" x2="21.3078" y2="3.3302" width="0.2032" layer="1"/>
@@
 <contactref element="R16" pad="2"/>
 <contactref element="R17" pad="2"/>
-<contactref element="U$57" pad="EN"/>
+<contactref element="LDO2" pad="EN"/>
 <wire x1="20.289" y1="2.54" x2="20.8224" y2="2.0066" width="0.2032" layer="1"/>
 <wire x1="20.8224" y1="2.0066" x2="21.0114" y2="2.0066" width="0.2032" layer="1"/>
